Commit message: Added base joint trying to avoid errors, looking ways for fixing gazebo

File: install/scara/share/scara/urdf/description.xacro (robot description, xacro)
@@ -6,4 +6,6 @@
   name="ros2Model">
   <link
+    name="world" />
+  <link
     name="base_link">
     <inertial>
@@ -36,4 +38,15 @@
     </visual>
   </link>
+  <joint
+    name="world_to_base"
+    type="fixed">
+    <parent
+      link="world" />
+    <child
+      link="base_link" />
+    <origin
+      xyz="0 0 0"
+      rpy="0 0 0" />
+  </joint>
   <link
     name="riel">
@@ -186,5 +199,5 @@
   </link>
   <joint
-    name="pendulo"
+    name="pendulo_joint"
     type="revolute">
     <origin

File: install/scara_gz/share/scara_gz/urdf/gz.xacro (robot description, xacro)
@@ -19,5 +19,5 @@
             <state_interface name="effort" />
         </joint>
-        <joint name="pendulo">
+        <joint name="pendulo_joint">
             <command_interface name="position">
                 <param name="min">-3.1416</param>
@@ -38,6 +38,5 @@
         </plugin>
         <!-- Physics parameters -->
-        <gravity>true</gravity>
-        <physics name="default_physics" default="true" type="ode">
+        <physics type="ode">
             <max_step_size>0.001</max_step_size>
             <real_time_factor>1.0</real_time_factor>
@@ -65,5 +64,4 @@
     <gazebo reference="base_link">
         <material>Gazebo/Grey</material>
-        <gravity>true</gravity>
         <mu1>0.2</mu1>
         <mu2>0.2</mu2>
@@ -73,5 +71,4 @@
     <gazebo reference="riel">
         <material>Gazebo/Blue</material>
-        <gravity>true</gravity>
         <mu1>0.2</mu1>
         <mu2>0.2</mu2>
@@ -81,5 +78,4 @@
     <gazebo reference="carro">
         <material>Gazebo/Blue</material>
-        <gravity>true</gravity>
         <mu1>0.2</mu1>
         <mu2>0.2</mu2>
@@ -89,5 +85,4 @@
     <gazebo reference="pendulo">
         <material>Gazebo/Blue</material>
-        <gravity>true</gravity>
         <mu1>0.2</mu1>
         <mu2>0.2</mu2>
@@ -97,16 +92,24 @@
     <!-- Gazebo specific properties for joints -->
     <gazebo reference="corredera">
-        <implicitSpringDamper>true</implicitSpringDamper>
-        <stopCfm>0.1</stopCfm>
-        <stopErp>0.2</stopErp>
-        <friction>0.1</friction>
-        <damping>0.1</damping>
+        <physics>
+            <ode>
+                <implicit_spring_damper>true</implicit_spring_damper>
+                <cfm>0.1</cfm>
+                <erp>0.2</erp>
+                <mu>0.1</mu>
+                <damping>0.1</damping>
+            </ode>
+        </physics>
     </gazebo>
-    <gazebo reference="pendulo">
-        <implicitSpringDamper>true</implicitSpringDamper>
-        <stopCfm>0.1</stopCfm>
-        <stopErp>0.2</stopErp>
-        <friction>0.1</friction>
-        <damping>0.1</damping>
+    <gazebo reference="pendulo_joint">
+        <physics>
+            <ode>
+                <implicit_spring_damper>true</implicit_spring_damper>
+                <cfm>0.1</cfm>
+                <erp>0.2</erp>
+                <mu>0.1</mu>
+                <damping>0.1</damping>
+            </ode>
+        </physics>
     </gazebo>
 </robot>

File: scara/urdf/description.xacro (robot description, xacro)
@@ -6,4 +6,6 @@
   name="ros2Model">
   <link
+    name="world" />
+  <link
     name="base_link">
     <inertial>
@@ -36,4 +38,15 @@
     </visual>
   </link>
+  <joint
+    name="world_to_base"
+    type="fixed">
+    <parent
+      link="world" />
+    <child
+      link="base_link" />
+    <origin
+      xyz="0 0 0"
+      rpy="0 0 0" />
+  </joint>
   <link
     name="riel">
@@ -186,5 +199,5 @@
   </link>
   <joint
-    name="pendulo"
+    name="pendulo_joint"
     type="revolute">
     <origin

Commit message: Gazebo not working yet

File: install/scara/share/scara/urdf/description.xacro (robot description, xacro)
@@ -199,5 +199,5 @@
   </link>
   <joint
-    name="pendulo_joint"
+    name="pendulo"
     type="revolute">
     <origin
@@ -213,5 +213,5 @@
       lower="-3.1416"
       upper="3.1416"
-      effort="10"
+      effort="0"
       velocity="10" />
   </joint>

File: install/scara_gz/share/scara_gz/urdf/gz.xacro (robot description, xacro)
@@ -19,9 +19,5 @@
             <state_interface name="effort" />
         </joint>
-        <joint name="pendulo_joint">
-            <command_interface name="position">
-                <param name="min">-3.1416</param>
-                <param name="max">3.1416</param>
-            </command_interface>
+        <joint name="pendulo">
             <state_interface name="position">
                 <param name="initial_value">0</param>
@@ -102,5 +98,5 @@
         </physics>
     </gazebo>
-    <gazebo reference="pendulo_joint">
+    <gazebo reference="pendulo">
         <physics>
             <ode>
