Commit message: Trying to work with both folders running

File: install/scara_gz/share/scara_gz/urdf/gz.xacro (robot description, xacro)
@@ -62,3 +62,51 @@
         </plugin>
     </gazebo>
+    <!-- Gazebo specific properties for links -->
+    <gazebo reference="base_link">
+        <material>Gazebo/Grey</material>
+        <gravity>true</gravity>
+        <mu1>0.2</mu1>
+        <mu2>0.2</mu2>
+        <kp>1000000.0</kp>
+        <kd>1.0</kd>
+    </gazebo>
+    <gazebo reference="riel">
+        <material>Gazebo/Blue</material>
+        <gravity>true</gravity>
+        <mu1>0.2</mu1>
+        <mu2>0.2</mu2>
+        <kp>1000000.0</kp>
+        <kd>1.0</kd>
+    </gazebo>
+    <gazebo reference="carro">
+        <material>Gazebo/Blue</material>
+        <gravity>true</gravity>
+        <mu1>0.2</mu1>
+        <mu2>0.2</mu2>
+        <kp>1000000.0</kp>
+        <kd>1.0</kd>
+    </gazebo>
+    <gazebo reference="pendulo">
+        <material>Gazebo/Blue</material>
+        <gravity>true</gravity>
+        <mu1>0.2</mu1>
+        <mu2>0.2</mu2>
+        <kp>1000000.0</kp>
+        <kd>1.0</kd>
+    </gazebo>
+    <!-- Gazebo specific properties for joints -->
+    <gazebo reference="corredera">
+        <implicitSpringDamper>true</implicitSpringDamper>
+        <stopCfm>0.1</stopCfm>
+        <stopErp>0.2</stopErp>
+        <friction>0.1</friction>
+        <damping>0.1</damping>
+    </gazebo>
+    <gazebo reference="pendulo">
+        <implicitSpringDamper>true</implicitSpringDamper>
+        <stopCfm>0.1</stopCfm>
+        <stopErp>0.2</stopErp>
+        <friction>0.1</friction>
+        <damping>0.1</damping>
+    </gazebo>
 </robot>

Commit message: GZ shows the model

File: install/scara_gz/share/scara_gz/urdf/gz.xacro (robot description, xacro)
@@ -71,4 +71,20 @@
         <kp>1000000.0</kp>
         <kd>1.0</kd>
+        <visual>
+            <geometry>
+                <mesh>
+                    <uri>package://scara/meshes/riel.STL</uri>
+                    <scale>1 1 1</scale>
+                </mesh>
+            </geometry>
+        </visual>
+        <collision>
+            <geometry>
+                <mesh>
+                    <uri>package://scara/meshes/riel.STL</uri>
+                    <scale>1 1 1</scale>
+                </mesh>
+            </geometry>
+        </collision>
     </gazebo>
     <gazebo reference="carro">
@@ -78,4 +94,20 @@
         <kp>1000000.0</kp>
         <kd>1.0</kd>
+        <visual>
+            <geometry>
+                <mesh>
+                    <uri>package://scara/meshes/carro.STL</uri>
+                    <scale>1 1 1</scale>
+                </mesh>
+            </geometry>
+        </visual>
+        <collision>
+            <geometry>
+                <mesh>
+                    <uri>package://scara/meshes/carro.STL</uri>
+                    <scale>1 1 1</scale>
+                </mesh>
+            </geometry>
+        </collision>
     </gazebo>
     <gazebo reference="pendulo">
@@ -85,4 +117,20 @@
         <kp>1000000.0</kp>
         <kd>1.0</kd>
+        <visual>
+            <geometry>
+                <mesh>
+                    <uri>package://scara/meshes/pendulo.STL</uri>
+                    <scale>1 1 1</scale>
+                </mesh>
+            </geometry>
+        </visual>
+        <collision>
+            <geometry>
+                <mesh>
+                    <uri>package://scara/meshes/pendulo.STL</uri>
+                    <scale>1 1 1</scale>
+                </mesh>
+            </geometry>
+        </collision>
     </gazebo>
     <!-- Gazebo specific properties for joints -->
