Commit message: Davinson borró

File: scara/urdf/description.xacro (robot description, xacro)
@@ -46,5 +46,5 @@
       link="base_link" />
     <origin
-      xyz="0 0 0"
+      xyz="0 0 1"
       rpy="0 0 0" />
   </joint>
@@ -159,5 +159,5 @@
   </joint>
   <link
-    name="pendulo">
+    name="pendulum_link">
     <inertial>
       <origin
@@ -199,5 +199,5 @@
   </link>
   <joint
-    name="pendulo"
+    name="pendulum_joint"
     type="revolute">
     <origin
@@ -207,5 +207,5 @@
       link="carro" />
     <child
-      link="pendulo" />
+      link="pendulum_link" />
     <axis
       xyz="0 0 -1" />

File: scara_gz/urdf/gz.xacro (robot description, xacro)
@@ -19,5 +19,5 @@
             <state_interface name="effort" />
         </joint>
-        <joint name="pendulo">
+        <joint name="pendulum_joint">
             <state_interface name="position">
                 <param name="initial_value">0</param>
@@ -111,5 +111,5 @@
         </collision>
     </gazebo>
-    <gazebo reference="pendulo">
+    <gazebo reference="pendulum_link">
         <material>Gazebo/Blue</material>
         <mu1>0.2</mu1>
@@ -146,5 +146,5 @@
         </physics>
     </gazebo>
-    <gazebo reference="pendulo">
+    <gazebo reference="pendulum_joint">
         <physics>
             <ode>
